File: mustache_pin/mustache_pin/mustache_pin.kicad_sch (KiCad schematic)
At the start: 8 parts, among them SW1 SW_SPDT

Commit message: silkscreens are weird
Connections:
- net at R1.2, R2.2, R3.2: now also SW1.3 (C); no longer SW1.1 (A)
Changed lines of the file:
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@@
     (stroke (width 0) (type default) (color 0 0 0 0))
   )
-  (symbol (lib_id "Switch:SW_SPDT") (at 66.04 74.93 0) (unit 1)
+  (symbol (lib_id "Switch:SW_SPDT") (at 66.04 74.93 0) (mirror x) (unit 1)
     (in_bom yes) (on_board yes) (fields_autoplaced)
     (property "Reference" "SW1" (id 0) (at 66.04 67.31 0))
